Commit message: Hoof included in the second goat model

File: NI_simulations/second_goat/second_goat_description/urdf/base/second_goat_base.xacro (robot description, xacro)
@@ -13,5 +13,5 @@
         <origin xyz="0 0 0" rpy="0 0 0" />
         <geometry>
-            <box size="${base_length} ${base_width} ${base_height}"/>
+            <box size="${base_body_length} ${base_body_width} ${base_body_height}"/>
         </geometry>
       </visual>
@@ -19,10 +19,10 @@
         <origin xyz="0 0 0" rpy="0 0 0" />
         <geometry>
-            <box size="${base_length} ${base_width} ${base_height}"/>
+            <box size="${base_body_length} ${base_body_width} ${base_body_height}"/>
         </geometry>
       </collision>
       <inertial>
-        <mass value="${base_mass}"/>
-        <inertia ixx="${base_mass*(base_width*base_width+base_height*base_height)/12}" ixy="0.0" ixz="0.0" iyy="${base_mass*(base_length*base_length+base_height*base_height)/12}" iyz="0.0" izz="${base_mass*(base_length*base_length+base_width*base_width)/12}"/>
+        <mass value="${base_body_mass}"/>
+        <inertia ixx="${base_body_mass*(base_body_width*base_body_width+base_body_height*base_body_height)/12}" ixy="0.0" ixz="0.0" iyy="${base_body_mass*(base_body_length*base_body_length+base_body_height*base_body_height)/12}" iyz="0.0" izz="${base_body_mass*(base_body_length*base_body_length+base_body_width*base_body_width)/12}"/>
       </inertial>
     </link>

File: NI_simulations/second_goat/second_goat_description/urdf/leg/hip_base/second_goat_hip_base.xacro (robot description, xacro)
@@ -3,14 +3,14 @@
   <xacro:macro name="hip_base" params="leg">
       <xacro:if value="${leg == 'RF'}">
-        <xacro:property name="origin_xyz_hip" value="${base_length/2-0.033} ${base_width/2-0.033} ${-base_height/2}"/>
+        <xacro:property name="origin_xyz_hip" value="${base_body_length/2-0.033} ${base_body_width/2-0.033} ${-base_body_height/2}"/>
       </xacro:if>
       <xacro:if value="${leg == 'LF'}">
-        <xacro:property name="origin_xyz_hip" value="${-base_length/2+0.033} ${base_width/2-0.033} ${-base_height/2}"/>
+        <xacro:property name="origin_xyz_hip" value="${-base_body_length/2+0.033} ${base_body_width/2-0.033} ${-base_body_height/2}"/>
       </xacro:if>
       <xacro:if value="${leg == 'RH'}">
-        <xacro:property name="origin_xyz_hip" value="${base_length/2 -0.033} ${-base_width/2+0.033} ${-base_height/2}"/>
+        <xacro:property name="origin_xyz_hip" value="${base_body_length/2 -0.033} ${-base_body_width/2+0.033} ${-base_body_height/2}"/>
       </xacro:if>
       <xacro:if value="${leg == 'LH'}">
-        <xacro:property name="origin_xyz_hip" value="${-base_length/2+0.033} ${-base_width/2+0.033} ${-base_height/2}"/>
+        <xacro:property name="origin_xyz_hip" value="${-base_body_length/2+0.033} ${-base_body_width/2+0.033} ${-base_body_height/2}"/>
       </xacro:if>
       <joint name="${leg}_base" type="fixed">
