Commit message: Another DoF added in the hoof

File: NI_simulations/second_goat/second_goat_description/urdf_hoof/hoof/claw/claw.xacro (robot description, xacro)
@@ -52,42 +52,4 @@
   </link>
 </xacro:if>
-  <!-- <link name="${side}_claw">
-    <visual>
-      <origin xyz="${claw_origin_xyz}" rpy="0 0 0" />
-      <geometry>
-          <box size="${claw_length} ${claw_width} ${claw_height}"/>
-      </geometry>
-    </visual>
-    <collision>
-      <origin xyz="${claw_origin_xyz}" rpy="0 0 0" />
-      <geometry>
-          <box size="${claw_length} ${claw_width} ${claw_height}"/>
-      </geometry>
-    </collision>
-    <inertial>
-      <mass value="${claw_mass}"/>
-      <origin xyz="${claw_origin_xyz}" rpy="0 0 0" />
-      <inertia ixx="${claw_mass*(claw_width*claw_width+claw_height*claw_height)/12}" ixy="0.0" ixz="0.0" iyy="${claw_mass*(claw_length*claw_length+claw_height*claw_height)/12}" iyz="0.0" izz="${claw_mass*(claw_length*claw_length+claw_width*claw_width)/12}"/>
-    </inertial>
-  </link>  -->
-  <!-- <link name="${side}_claw">
-    <visual>
-      <origin xyz="0.06 -0.025 0.005" rpy="${-pi/2} 0 ${pi/2}" />
-      <geometry>
-          <mesh filename="${mesh_claw}" scale="0.0015 0.0015 0.0015" />
-      </geometry>
-    </visual>
-    <collision>
-      <origin xyz="0.06 -0.025 0.005" rpy="${-pi/2} 0 ${pi/2}" />
-      <geometry>
-          <mesh filename="${mesh_claw}" scale="0.0015 0.0015 0.0015" />
-      </geometry>
-    </collision>
-    <inertial>
-      <mass value="${claw_mass}"/>
-      <origin xyz="${claw_origin_xyz}" rpy="0 0 0" />
-      <inertia ixx="${claw_mass*(claw_width*claw_width+claw_height*claw_height)/12}" ixy="0.0" ixz="0.0" iyy="${claw_mass*(claw_length*claw_length+claw_height*claw_height)/12}" iyz="0.0" izz="${claw_mass*(claw_length*claw_length+claw_width*claw_width)/12}"/>
-    </inertial>
-  </link> -->
 <gazebo reference="${leg}_${side}_claw">
         <material>Gazebo/WoodFloor</material>

File: NI_simulations/second_goat/second_goat_description/urdf_hoof/hoof/coffin_joint/coffin_joint.xacro (robot description, xacro)
@@ -18,9 +18,9 @@
       <dynamics damping="0.07" friction="0" />
     </joint>
-    <gazebo reference="joint_${side}_coffin_${leg}">
+<gazebo reference="joint_${side}_coffin_${leg}">
   <implicitSpringDamper>True</implicitSpringDamper>
 </gazebo>
   <gazebo>
-        <plugin name="${side}_sea_j2" filename="libsea_plugin.so">
+        <plugin name="${side}_sea_j5" filename="libsea_plugin.so">
             <joint>joint_${side}_coffin_${leg}</joint>
             <namespace>goat_robot</namespace>

File: NI_simulations/second_goat/second_goat_description/urdf_hoof/hoof/hoof.xacro (robot description, xacro)
@@ -3,4 +3,10 @@
   <!-- Leg components -->
   <xacro:macro name="hoof" params="leg side" >
+    <!-- Fetlock Joint -->
+    <xacro:include filename="$(find second_goat_description)/urdf_hoof/hoof/fetlock_joint/fetlock_joint.xacro"/>
+    <xacro:fetlock_joint leg="${leg}" side="${side}" />
+    <!-- Declaw Link -->
+    <xacro:include filename="$(find second_goat_description)/urdf_hoof/hoof/declaw/declaw.xacro"/>
+    <xacro:declaw leg="${leg}" side="${side}"/>
     <!-- Pastern Joint -->
     <xacro:include filename="$(find second_goat_description)/urdf_hoof/hoof/pastern_joint/pastern_joint.xacro"/>

File: NI_simulations/second_goat/second_goat_description/urdf_hoof/hoof/pastern_joint/pastern_joint.xacro (robot description, xacro)
@@ -3,19 +3,19 @@
   <xacro:macro name="pastern_joint" params="leg side">
   <xacro:if value="${side == 'R'}">
-    <xacro:property name="pastern_origin_xyz" value="0 ${base_radius/2} 0"/>
+    <xacro:property name="pastern_origin_xyz" value="0 0 0"/>
   </xacro:if>
   <xacro:if value="${side == 'L'}">
-    <xacro:property name="pastern_origin_xyz" value="0 ${-base_radius/2} 0"/>
+    <xacro:property name="pastern_origin_xyz" value="0 0 0"/>
   </xacro:if>
     <joint name="joint_${side}_pastern_${leg}" type="prismatic">
-      <parent link="base_link_hoof_${leg}"/>
+      <parent link="${leg}_${side}_declaw"/>
       <child link="${leg}_${side}_phalange"/>
-      <origin xyz="${pastern_origin_xyz}" rpy="0 0 0" />
+      <origin xyz="${pastern_origin_xyz}" rpy="0 ${-pi/2} 0" />
       <axis xyz="0 0 1" />
       <limit effort="30" velocity="1.0" lower="-0.02" upper="0.02" />
-      <dynamics damping="0.7" friction="0" />
+      <dynamics damping="50.0" friction="0" />
     </joint>
   <gazebo>
-      <plugin name="${side}_sea_j1" filename="libsea_plugin.so">
+      <plugin name="${side}_sea_j4" filename="libsea_plugin.so">
           <joint>joint_${side}_pastern_${leg}</joint>
           <namespace>goat_robot</namespace>

File: NI_simulations/second_goat/second_goat_description/urdf_hoof/metacarpus/metacarpus.xacro (robot description, xacro)
@@ -1,5 +1,5 @@
 <?xml version='1.0'?>
 <robot name="goat_robot" xmlns:xacro="http://www.ros.org/wiki/xacro">
-<xacro:macro name="metacarpus" params="name leg" >
+<xacro:macro name="metacarpus" params="leg" >
   <!-- <link name="world">
   </link>  -->
@@ -7,7 +7,7 @@
         <origin xyz="0 -0.076 0" rpy="${-pi/2} 0 0"/>
         <parent link="${leg}_shank"/>
-        <child link="${name}_${leg}"/>
+        <child link="metacarpus_${leg}"/>
   </joint>
-  <link name="${name}_${leg}">
+  <link name="metacarpus_${leg}">
       <visual>
         <origin xyz="0 0 0" rpy="0 0 0" />
@@ -28,5 +28,5 @@
       </inertial>
   </link>
-  <gazebo reference="${name}_${leg}">
+  <gazebo reference="metacarpus_${leg}">
         <material>Gazebo/WoodFloor</material>
   </gazebo>
